File: Premium lumpen.kicad_sch (KiCad schematic)
At the start: 138 parts, among them J1 Conn_01x04_MountingPin, J2 AVR-ISP-6, SW1 SW_Push, SW2 RotaryEncoder_Switch, SW3 RotaryEncoder_Switch, U1 ATmega32U4-M, Y1 Crystal_GND24_Small

Commit message: changed zone filling on lumpen, worked on premium
Parts:
- removed Drgb6: WS2812-2020, CrumpPrints:WS2812-2020, symbol crumpschemes:WS2812-2020
- added D6, D7, D8, D9: D_Small, Keebio-Parts:D_SOD123F, symbol Device:D_Small
- added Drgb2: WS2812-2020, Keebio-Parts:SK6812-MINI-E, symbol crumpschemes:WS2812-2020
- added MX46, MX47, MX48, MX49: MX-NoLED, MX_Only:MXOnly-1U-NoLED, symbol MX_Alps_Hybrid:MX-NoLED
- added SW4, SW5: RotaryEncoder_Switch, Keebio-Parts:RotaryEncoder_EC11-no-legs, symbol Device:RotaryEncoder_Switch
- D24: footprint Diode_SMD:D_0402_1005Metric -> Keebio-Parts:D_SOD123F
- Drgb1, Drgb3, Drgb4: footprint CrumpPrints:WS2812-2020 -> Keebio-Parts:SK6812-MINI-E
- J2: footprint Keebio-Parts:ICSP-Header -> Keebio-Parts:ICSP_1.27mm
Connections:
- net  ROW3: now also D9.1 (K); no longer D16.3 (K), D24.1 (K), D31.3 (K), D42.3 (K), D5.3 (K)
- net COL0: now also SW3.S2, MX46.1 (COL), MX47.1 (COL), MX48.1 (COL), MX49.1 (COL), SW4.S2, SW5.S2; no longer MX1.1 (COL), MX13.1 (COL), MX25.1 (COL), MX37.1 (COL)
- net COL1: now also MX1.1 (COL), MX13.1 (COL), MX25.1 (COL), MX37.1 (COL); no longer MX14.1 (COL), MX2.1 (COL), MX26.1 (COL), MX38.1 (COL)
- net COL10: now also MX10.1 (COL), MX22.1 (COL), MX34.1 (COL); no longer MX11.1 (COL), MX23.1 (COL), MX35.1 (COL), MX44.1 (COL), SW3.S2
- net COL11: now also MX11.1 (COL), MX23.1 (COL), MX35.1 (COL), MX44.1 (COL); no longer MX12.1 (COL), MX24.1 (COL), MX36.1 (COL), MX45.1 (COL)
- net COL2: now also MX14.1 (COL), MX2.1 (COL), MX26.1 (COL), MX38.1 (COL); no longer MX15.1 (COL), MX27.1 (COL), MX3.1 (COL)
- net COL3: now also MX15.1 (COL), MX27.1 (COL), MX3.1 (COL), U1.1 (PE6); no longer MX16.1 (COL), MX28.1 (COL), MX39.1 (COL), MX4.1 (COL)
- net COL4: now also MX16.1 (COL), MX28.1 (COL), MX39.1 (COL), MX4.1 (COL); no longer MX17.1 (COL), MX29.1 (COL), MX40.1 (COL), MX5.1 (COL)
- net COL5: now also MX17.1 (COL), MX29.1 (COL), MX40.1 (COL), MX5.1 (COL); no longer MX18.1 (COL), MX30.1 (COL), MX41.1 (COL), MX6.1 (COL)
- net COL6: now also MX18.1 (COL), MX30.1 (COL), MX41.1 (COL), MX6.1 (COL); no longer MX19.1 (COL), MX31.1 (COL), MX7.1 (COL)
- net COL7: now also MX19.1 (COL), MX31.1 (COL), MX7.1 (COL); no longer MX20.1 (COL), MX32.1 (COL), MX42.1 (COL), MX8.1 (COL)
- net COL8: now also MX20.1 (COL), MX32.1 (COL), MX42.1 (COL), MX8.1 (COL); no longer MX21.1 (COL), MX33.1 (COL), MX43.1 (COL), MX9.1 (COL)
- net COL9: now also MX21.1 (COL), MX33.1 (COL), MX43.1 (COL), MX9.1 (COL); no longer MX10.1 (COL), MX22.1 (COL), MX34.1 (COL)
- net GND: now also Drgb2.2 (VSS), SW4.C, SW5.C
- net RGB_per key: now also U1.41 (PF0); no longer U1.40 (PF1)
- net ROTARY_A: now also SW4.A; no longer SW2.A
- net ROTARY_B: now also SW4.B; no longer SW2.B
- net ROTARY_C: now also SW2.A; no longer SW3.A
- net ROTARY_D: now also SW2.B; no longer SW3.B
- net ROW0: now also D6.1 (K)
- net ROW1: now also D7.1 (K)
- net ROW2: now also D8.1 (K)
- net VCC: now also Drgb2.4 (VDD)
- net at D42.1 (A), MX44.2 (ROW): no longer SW3.S1
- net at Drgb49.1 (DOUT): now also Drgb9.3 (DIN)
- net at D2.1 (A), MX1.2 (ROW): no longer SW2.S1
- net at Drgb3.3 (DIN): now also Drgb2.1 (DOUT); no longer Drgb1.1 (DOUT)
- net at Drgb51.1 (DOUT): now also Drgb1.3 (DIN)
- removed net RGB_Underglow: Drgb1.3 (DIN), U1.41 (PF0)
- new net: D16.3 (K), D24.1 (K), D31.3 (K), D42.3 (K), D5.3 (K)
- new net: D6.2 (A), MX46.2 (ROW), SW4.S1
- new net: D9.2 (A), MX49.2 (ROW), SW3.S1
- new net: D8.2 (A), MX48.2 (ROW), SW5.S1
- new net: D7.2 (A), MX47.2 (ROW), SW2.S1
- new net: Drgb1.1 (DOUT), Drgb2.3 (DIN)
- new net COL12: MX12.1 (COL), MX24.1 (COL), MX36.1 (COL), MX45.1 (COL), U1.40 (PF1)
- new net ROTARY_E: SW5.A
- new net ROTARY_F: SW5.B
- new net ROTARY_G: SW3.A
- new net ROTARY_H: SW3.B
- no-connect marks 0 -> 1
Other:
- moved on the sheet: D10, D11, D12, D16, D17, D18, D19, D2, D24, D25, D26, D27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

Commit message: premium 3 flex cut matrix routed
Parts:
- Drgb1, Drgb10, Drgb11, Drgb12, Drgb13, Drgb14, Drgb15, Drgb16, Drgb17, Drgb18, Drgb19, Drgb2, Drgb20, Drgb21, Drgb22, Drgb23, Drgb24, Drgb25, Drgb26, Drgb27, Drgb28, Drgb29, Drgb3, Drgb30, Drgb31, Drgb32, Drgb33, Drgb34, Drgb35, Drgb36, Drgb37, Drgb38, Drgb39, Drgb4, Drgb40, Drgb41, Drgb42, Drgb43, Drgb44, Drgb45, Drgb46, Drgb47, Drgb48, Drgb49, Drgb50, Drgb51, Drgb7, Drgb8, Drgb9: footprint Keebio-Parts:SK6812-MINI-E -> CrumpPrints:WS2812-2020

Commit message: auto save
Connections:
- net  ROW3: now also D16.3 (K), D24.1 (K), D31.3 (K), D42.3 (K), D5.3 (K)
Changed lines of the file:
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@@
   (junction (at 238.125 109.982) (diameter 0) (color 0 0 0 0)
   )
+  (junction (at 149.225 109.982) (diameter 0) (color 0 0 0 0)
+  )
   (junction (at 200.025 57.15) (diameter 0) (color 0 0 0 0)
   )
@@
   )
   (junction (at 381.381 102.235) (diameter 0) (color 0 0 0 0)
-  )
-  (junction (at 149.225 109.982) (diameter 0) (color 0 0 0 0)
   )
   (junction (at 250.825 74.93) (diameter 0) (color 0 0 0 0)
@@
     (stroke (width 0) (type default) (color 0 0 0 0))
   )
-  (wire (pts (xy 135.255 109.982) (xy 149.225 109.982))
-    (stroke (width 0) (type default) (color 0 0 0 0))
-  )
   (wire (pts (xy 50.546 28.321) (xy 50.546 30.861))
     (stroke (width 0) (type default) (color 0 0 0 0))
@@
     (stroke (width 0) (type default) (color 0 0 0 0))
   )
-  (wire (pts (xy 131.699 109.982) (xy 135.128 109.982))
+  (wire (pts (xy 131.699 109.982) (xy 149.225 109.982))
     (stroke (width 0) (type default) (color 0 0 0 0))
   )
@@
     (stroke (width 0) (type default) (color 0 0 0 0))
   )
+  (wire (pts (xy 149.225 109.982) (xy 189.865 109.982))
+    (stroke (width 0) (type default) (color 0 0 0 0))
+  )
   (wire (pts (xy 138.049 64.77) (xy 136.779 64.77))
     (stroke (width 0) (type default) (color 0 0 0 0))
@@
     (stroke (width 0) (type default) (color 0 0 0 0))
   )
-  (wire (pts (xy 149.225 109.982) (xy 189.865 109.982))
-    (stroke (width 0) (type default) (color 0 0 0 0))
-  )

Commit message: premium work
Parts:
- Drgb1, Drgb10, Drgb11, Drgb12, Drgb13, Drgb14, Drgb15, Drgb16, Drgb17, Drgb18, Drgb19, Drgb2, Drgb20, Drgb21, Drgb22, Drgb23, Drgb24, Drgb25, Drgb26, Drgb27, Drgb28, Drgb29, Drgb3, Drgb30, Drgb31, Drgb32, Drgb33, Drgb34, Drgb35, Drgb36, Drgb37, Drgb38, Drgb39, Drgb4, Drgb40, Drgb41, Drgb42, Drgb43, Drgb44, Drgb45, Drgb46, Drgb47, Drgb48, Drgb49, Drgb50, Drgb51, Drgb7, Drgb8, Drgb9: footprint CrumpPrints:WS2812-2020 -> Keebio-Parts:SK6812-MINI-E
