File: lumpen.kicad_sch (KiCad schematic)
At the start: 93 parts, among them J1 Conn_01x03, SW1 RotaryEncoder_Switch

Commit message: lumpen v1.1
changed the placement of microcontroller ever so slightly for hopefully better fitment for switch

added rotary legs for better support of lowprofile non click rotaries
Parts:
- SW1: footprint Keebio-Parts:RotaryEncoder_EC11-no-legs -> Keebio-Parts:RotaryEncoder_EC11
Changed lines of the file:
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@@
     (property "Reference" "SW1" (id 0) (at 258.064 84.836 0))
     (property "Value" "RotaryEncoder_Switch" (id 1) (at 258.064 87.376 0))
-    (property "Footprint" "Keebio-Parts:RotaryEncoder_EC11-no-legs" (id 2) (at 261.874 99.06 0)
+    (property "Footprint" "Keebio-Parts:RotaryEncoder_EC11" (id 2) (at 261.874 99.06 0)
       (effects (font (size 1.27 1.27)) hide)
     )
@@
     )
     (path "/73532d33-fe03-43bd-8e2a-c27b234769f0"
-      (reference "SW1") (unit 1) (value "RotaryEncoder_Switch") (footprint "Keebio-Parts:RotaryEncoder_EC11-no-legs")
-    )
-  )
+      (reference "SW1") (unit 1) (value "RotaryEncoder_Switch") (footprint "Keebio-Parts:RotaryEncoder_EC11")
+    )
+  )
